File: badgelife_dev_board.kicad_pcb (KiCad board)
At the start: 2 copper layers, 33 x 42 mm, 14 parts, among them J1 Conn_01x08, J2 Conn_01x08, J3 Conn_01x09, J4 Conn_01x09, X1 Badgelife_shitty_connector

Commit message: work in progress
Other:
- board size 33 x 42 mm -> 33.2 x 42.2 mm
Changed lines of the file:
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@@
-(kicad_pcb (version 4) (host pcbnew 4.0.7-e2-6376~61~ubuntu18.04.1)
+(kicad_pcb (version 4) (host pcbnew 4.0.6+dfsg1-1)
   (general
-    (links 0)
+    (links 34)
     (no_connects 0)
-    (area 103.249999 137.5 153.750001 188.750001)
+    (area 94.116316 137.5 153.750001 188.750001)
     (thickness 1.6)
-    (drawings 28)
+    (drawings 37)
     (tracks 55)
     (zones 0)
@@
     (add_net SDA)
   )
+  (module mrmeeseeks:Badgelife-Shitty-2x2 (layer F.Cu)
+    (at 128.5 179.5)
+    (descr "Through hole angled pin header, 2x02, 2.54mm pitch, 6mm pin length, double rows")
+    (tags "Through hole angled pin header THT 2x02 2.54mm double row")
+    (fp_text reference X1 (at 0 0) (layer F.Fab)
+      (effects (font (size 1 1) (thickness 0.15)))
+    )
+    (fp_text value Badgelife_shitty_connector (at 0 4.2) (layer F.Fab)
+      (effects (font (size 1 1) (thickness 0.15)))
+    )
+    (fp_text user sda (at 3.5 -1.5) (layer F.SilkS)
+      (effects (font (size 0.7 0.7) (thickness 0.1)))
+    )
+    (fp_line (start -25 9) (end 25 9) (layer F.Fab) (width 0.1))
+    (fp_circle (center -2.54 -2.54) (end -2.14 -2.54) (layer F.SilkS) (width 0.15))
+    (fp_line (start -25 -41) (end -25 9) (layer F.Fab) (width 0.1))
+    (fp_line (start 25 -41) (end 25 9) (layer F.Fab) (width 0.1))
+    (fp_line (start -25 -41) (end 25 -41) (layer F.Fab) (width 0.1))
+    (fp_text user scl (at 3.25 2.25) (layer F.SilkS)
+      (effects (font (size 0.7 0.7) (thickness 0.1)))
+    )
+    (fp_text user gnd (at -3.25 2.25) (layer F.SilkS)
+      (effects (font (size 0.7 0.7) (thickness 0.1)))
+    )
+    (fp_text user 3.3v (at -3.5 -1.5) (layer F.SilkS)
+      (effects (font (size 0.7 0.7) (thickness 0.1)))
+    )
+    (pad 4 thru_hole circle (at 1.27 -1.27) (size 1.7 1.7) (drill 1) (layers *.Cu *.Mask)
+      (net 3 SDA))
+    (pad 3 thru_hole oval (at 1.27 1.27) (size 1.7 1.7) (drill 1) (layers *.Cu *.Mask)
+      (net 4 SCL))
+    (pad 1 thru_hole oval (at -1.27 -1.27) (size 1.7 1.7) (drill 1) (layers *.Cu *.Mask)
+      (net 1 +3V3))
+    (pad 2 thru_hole oval (at -1.27 1.27) (size 1.7 1.7) (drill 1) (layers *.Cu *.Mask)
+      (net 2 GND))
+  )
   (module mrmeeseeks:Pin_Header_Straight_2x09_Pitch2.54mm-NoSilk (layer F.Cu)
     (at 118.364 171.2 90)
@@
     (pad 17 thru_hole oval (at 0 20.32 90) (size 1.7 1.7) (drill 1) (layers *.Cu *.Mask))
     (pad 18 thru_hole oval (at 2.54 20.32 90) (size 1.7 1.7) (drill 1) (layers *.Cu *.Mask))
-  )
-  (module mrmeeseeks:Badgelife-Shitty-2x2 (layer F.Cu)
-    (at 128.5 179.5)
-    (descr "Through hole angled pin header, 2x02, 2.54mm pitch, 6mm pin length, double rows")
-    (tags "Through hole angled pin header THT 2x02 2.54mm double row")
-    (fp_text reference X1 (at 0 0) (layer F.Fab)
-      (effects (font (size 1 1) (thickness 0.15)))
-    )
-    (fp_text value Badgelife_shitty_connector (at 0 4.2) (layer F.Fab)
-      (effects (font (size 1 1) (thickness 0.15)))
-    )
-    (fp_text user sda (at 3.5 -1.5) (layer F.SilkS)
-      (effects (font (size 0.7 0.7) (thickness 0.1)))
-    )
-    (fp_line (start -25 9) (end 25 9) (layer F.Fab) (width 0.1))
-    (fp_circle (center -2.54 -2.54) (end -2.14 -2.54) (layer F.SilkS) (width 0.15))
-    (fp_line (start -25 -41) (end -25 9) (layer F.Fab) (width 0.1))
-    (fp_line (start 25 -41) (end 25 9) (layer F.Fab) (width 0.1))
-    (fp_line (start -25 -41) (end 25 -41) (layer F.Fab) (width 0.1))
-    (fp_text user scl (at 3.25 2.25) (layer F.SilkS)
-      (effects (font (size 0.7 0.7) (thickness 0.1)))
-    )
-    (fp_text user gnd (at -3.25 2.25) (layer F.SilkS)
-      (effects (font (size 0.7 0.7) (thickness 0.1)))
-    )
-    (fp_text user 3.3v (at -3.5 -1.5) (layer F.SilkS)
-      (effects (font (size 0.7 0.7) (thickness 0.1)))
-    )
-    (pad 4 thru_hole circle (at 1.27 -1.27) (size 1.7 1.7) (drill 1) (layers *.Cu *.Mask)
-      (net 3 SDA))
-    (pad 3 thru_hole oval (at 1.27 1.27) (size 1.7 1.7) (drill 1) (layers *.Cu *.Mask)
-      (net 4 SCL))
-    (pad 1 thru_hole oval (at -1.27 -1.27) (size 1.7 1.7) (drill 1) (layers *.Cu *.Mask)
-      (net 1 +3V3))
-    (pad 2 thru_hole oval (at -1.27 1.27) (size 1.7 1.7) (drill 1) (layers *.Cu *.Mask)
-      (net 2 GND))
   )
   (module mrmeeseeks:Power_Rail-01x08 (layer F.Cu)
@@
       (xy -0.777268 -2.713942) (xy -0.713043 -2.730292) (xy -0.650806 -2.707788)) (layer F.SilkS) (width 0.01))
   )
+  (gr_line (start 145.05 145.95) (end 145.05 144.8) (angle 90) (layer Edge.Cuts) (width 0.15))
+  (gr_line (start 116.8 141) (end 119.25 141) (angle 90) (layer Edge.Cuts) (width 0.15))
+  (gr_line (start 116.8 141) (end 118.1 141) (angle 90) (layer Edge.Cuts) (width 0.15))
+  (gr_line (start 111.9 145.45) (end 111.95 145.45) (angle 90) (layer Edge.Cuts) (width 0.15))
+  (gr_line (start 111.9 146) (end 111.9 145.45) (angle 90) (layer Edge.Cuts) (width 0.15))
+  (gr_line (start 138 183.1) (end 118.15 183.1) (angle 90) (layer Edge.Cuts) (width 0.15))
+  (gr_line (start 145 145.3) (end 145 144.8) (angle 90) (layer Edge.Cuts) (width 0.15))
+  (gr_line (start 111.95 145.7) (end 111.95 175.7) (angle 90) (layer Edge.Cuts) (width 0.15))
+  (gr_line (start 145 144.95) (end 145 177.25) (angle 90) (layer Edge.Cuts) (width 0.15))
+  (gr_arc (start 138.55 176.65) (end 145 177.2) (angle 90) (layer Edge.Cuts) (width 0.15))
+  (gr_line (start 111.9 175.65) (end 111.9 176.65) (angle 90) (layer Edge.Cuts) (width 0.15))
+  (gr_arc (start 118.4 176.6) (end 118.1 183.1) (angle 90) (layer Edge.Cuts) (width 0.15))
+  (gr_line (start 117.6 141.05) (end 140 141.05) (angle 90) (layer Edge.Cuts) (width 0.15))
+  (gr_arc (start 140.65 145.45) (end 139.95 141.05) (angle 90) (layer Edge.Cuts) (width 0.15))
+  (gr_arc (start 117.05 146.15) (end 111.9 145.55) (angle 90) (layer Edge.Cuts) (width 0.15))
   (dimension 6.500769 (width 0.3) (layer Dwgs.User)
     (gr_text "6.501 mm" (at 99.902029 145.192277 270.881404) (layer Dwgs.User)
@@
     (arrow2b (pts (xy 101.20187 141.92151) (xy 101.80555 143.03886)))
   )
-  (gr_line (start 145 176) (end 133 183) (layer Edge.Cuts) (width 0.15))
-  (gr_line (start 133 183) (end 124 183) (layer Edge.Cuts) (width 0.15))
-  (gr_line (start 112 176) (end 112 141) (layer Edge.Cuts) (width 0.15))
-  (gr_line (start 124 183) (end 112 176) (layer Edge.Cuts) (width 0.15))
-  (gr_line (start 145 141) (end 145 176) (layer Edge.Cuts) (width 0.15))
-  (gr_line (start 112 141) (end 145 141) (layer Edge.Cuts) (width 0.15))
   (dimension 27.2 (width 0.3) (layer Dwgs.User)
     (gr_text "27.200 mm" (at 128.5 138.85) (layer Dwgs.User)
@@
   (segment (start 117.5 176.25) (end 116.25 176.25) (width 0.6) (layer F.Cu) (net 1))
   (segment (start 119.48 178.23) (end 117.5 176.25) (width 0.6) (layer F.Cu) (net 1))
-  (segment (start 127.23 178.23) (end 119.48 178.23) (width 0.6) (layer F.Cu) (net 1))
   (segment (start 115.7986 171.196) (end 115.7986 168.656) (width 2.54) (layer F.Cu) (net 1))
   (segment (start 115.7986 166.116) (end 115.7986 168.656) (width 2.54) (layer F.Cu) (net 1))
@@
   (segment (start 115.7986 153.416) (end 115.7986 155.956) (width 2.54) (layer F.Cu) (net 1))
   (segment (start 115.7986 171.196) (end 115.7986 153.416) (width 2.54) (layer F.Cu) (net 1))
+  (segment (start 127.23 178.23) (end 119.48 178.23) (width 0.6) (layer F.Cu) (net 1))
+  (segment (start 127.23 180.77) (end 126.027919 180.77) (width 0.6) (layer B.Cu) (net 2))
   (segment (start 140 176.25) (end 141.224 175.026) (width 0.6) (layer B.Cu) (net 2))
   (segment (start 141.224 175.026) (end 141.224 171.196) (width 0.6) (layer B.Cu) (net 2))
@@
   (segment (start 125.75 180.5) (end 124.25 179) (width 0.6) (layer B.Cu) (net 2))
   (segment (start 125.757919 180.5) (end 125.75 180.5) (width 0.6) (layer B.Cu) (net 2))
-  (segment (start 127.23 180.77) (end 126.027919 180.77) (width 0.6) (layer B.Cu) (net 2))
   (segment (start 126.027919 180.77) (end 125.757919 180.5) (width 0.6) (layer B.Cu) (net 2))
   (segment (start 141.224 155.956) (end 141.224 153.416) (width 2.54) (layer F.Cu) (net 2))
@@
   (segment (start 134.75 177.25) (end 140.5 177.25) (width 0.6) (layer B.Cu) (net 3))
   (segment (start 133.77 178.23) (end 134.75 177.25) (width 0.6) (layer B.Cu) (net 3))
-  (segment (start 129.77 178.23) (end 133.77 178.23) (width 0.6) (layer B.Cu) (net 3))
   (segment (start 120.904 150.876) (end 118.364 150.876) (width 2.54) (layer F.Cu) (net 3))
   (segment (start 123.444 150.876) (end 120.904 150.876) (width 2.54) (layer F.Cu) (net 3))
@@
   (segment (start 136.144 150.876) (end 133.604 150.876) (width 2.54) (layer F.Cu) (net 3))
   (segment (start 138.684 150.876) (end 136.144 150.876) (width 2.54) (layer F.Cu) (net 3))
+  (segment (start 129.77 178.23) (end 133.77 178.23) (width 0.6) (layer B.Cu) (net 3))
   (segment (start 129.77 180.77) (end 133.604 176.936) (width 0.6) (layer F.Cu) (net 4))
   (segment (start 133.604 176.936) (end 133.604 173.736) (width 0.6) (layer F.Cu) (net 4))
