File: badgelife_dev_board.sch (KiCad schematic (older format))
At the start: 5 parts, among them J1 Conn_01x08, J2 Conn_01x08, J3 Conn_01x09, J4 Conn_01x09, X1 Badgelife_shitty_connector

Commit message: add badgelife add-on proto board for the SAO v1.69bis standard
Parts:
- added J5, J6: Conn_01x08, symbol badgelife_dev_board-rescue:Conn_01x08
- added J7: Conn_02x03_Odd_Even, badgelife_sao_v169bis:Badgelife-SAOv169-SAO-2x3, symbol Connector_Generic:Conn_02x03_Odd_Even
- added J8, J9: Conn_01x09, symbol badgelife_dev_board-rescue:Conn_01x09
- J1, J2: symbol Conn_01x08 -> badgelife_dev_board-rescue:Conn_01x08
- J3, J4: symbol Conn_01x09 -> badgelife_dev_board-rescue:Conn_01x09
- X1: symbol Badgelife_shitty_connector -> badgelife_dev_board-rescue:Badgelife_shitty_connector
Connections:
- net labels added: GPIO1, GPIO2
- wire segments 38 -> 138
